File: hardware/led-control.kicad_sch (KiCad schematic)
At the start: 21 parts, among them J401 ZX-XH2.54-3PWT, SW402 EC11J1525402, U402 TPS259531DSGR, U403 SN74LVC1T45DBVR

Commit message: feat: WIP pcb layout
Parts:
- added C408: 100n, Capacitor_SMD:C_0402_1005Metric, symbol Device:C
- added D401: SS34, Diode_SMD:D_SMA, symbol Device:D_Schottky
- added R414: 100k, Resistor_SMD:R_0402_1005Metric, symbol Device:R
- C404: Rotation Offset (none) -> 180
- J401: Position Offset (none) -> 0,-3.59
Connections:
- net +5V: now also D401.1 (K)
- net GND: now also C408.2, D401.2 (A)
- net EN_UVLO: now reaches R406.1, R407.1, U402.2 (EN_UVLO)
- net dVdt: now reaches C403.1, U402.1 (dVdt)
- net ILM: now reaches R403.1, U402.7 (ILM)
- net ILM: now also R414.1
- net CONN_LDATA: now reaches J401.2 (Pin_2), R409.2, R410.1
- net B_LDATA: now reaches R409.1, U403.4 (B)
- net LED_DATA renamed MCU_LDATA
- new net LED_ISENSE: C408.1, R414.2
Other:
- note added: "D401 clamps the negative spike on +5V when U402 trips into the LED cable inductance (TPS2595 transient protection)."
- note added: "Debounce A/B and the push button in firmware. A = GPIO3, B = GPIO2, push = GPIO6 (active low)."
- note added: "J401: 1 = switched +5V, 2 = DATA, 3 = GND. U403: DIR high selects A -> B. VCC isolation + Ioff prevent DATA from powering an unpowered LED chain. Fit C401 / C407 close to the two supply pins."
- note added: "R414 + C408: LED current monitor to GPIO0 (ADC1_CH0), use 0 dB atten. I_LED = V_ADC / (R403 x GIMON) = 3.62 A/V x V_ADC (GIMON 276 uA/A typ, 254..299). About 0.56 V at the 2.04 A limit. RC = 10 ms averages the pixel PWM ripple. R414 takes < 1 % of the ILM current, so ILIM is unchanged. Set GPIO0 to ADC (no pull) before enabling LED_PWR_EN."
- note removed: "Debounce A/B and the push button in firmware. A = GPIO19, B = GPIO20, push = GPIO21 (active low)."
- note removed: "J401: 1 = switched +5V, 2 = DATA, 3 = GND. U403: DIR high selects A -> B. VCC isolation + Ioff prevent DATA from powering an unpowered LED chain. Fit C406 / C407 close to the two supply pins."
- moved on the sheet: C401, C407, J401, R408, R409, R410, U403
