File: hardware/mcu.kicad_sch (KiCad schematic)
At the start: 18 parts, among them J201 USB_C_Receptacle_USB2.0, SW201 RESET, SW202 BOOT, U201 ESP32-C6-MINI-1-N4, U202 USBLC6-2SC6

Commit message: feat: Added led controller sheet
Parts:
- renumbered C201 to C301, C202 to C302, C203 to C303, C204 to C304, D302 to D301, J201 to J301, R201 to R301, R202 to R302, R203 to R303, R205 to R304, R204 to R305, R210 to R306, R206 to R307, R207 to R308, SW201 to SW301, SW202 to SW302, U201 to U301, U202 to U302
Connections:
- net ENC_A: now reaches U301.25 (IO19)
- net ENC_B: now reaches U301.26 (IO20)
- net ENC_SW_N: now reaches U301.27 (IO21)
- net LED_DATA: now reaches U301.28 (IO22)
- net LED_PWR_EN: now reaches U301.5 (IO2)
- net LED_FAULT_N: now reaches U301.6 (IO3)
- no-connect marks 18 -> 12
Other:
- note added: "Supply requirement: dedicated USB-C 5 V / 3 A. R206 / R207 provide Rd. No PD negotiation or current detection."
- title: (none) -> LED power and controls

Commit message: feat: WIP pcb layout
Parts:
- removed R304, R305: 2k2, Resistor_SMD:R_0402_1005Metric, symbol Device:R
- U301: value ESP32-C6-MINI-1-N4 -> ESP32-C6-MINI-1U-H4; footprint RF_Module:ESP32-C6-MINI-1 -> PCM_Espressif:ESP32-C6-MINI-1U; symbol RF_Module:ESP32-C6-MINI-1 -> PCM_Espressif:ESP32-C6-MINI-1/U; LCSC Part # C5736265 -> C20627095; Position Offset (none) -> 0,-2.68
Connections:
- net I2C_SDA is gone; now on net LED_FAULT_N: U301.13 (GPIO1/ADC1_CH1/XTAL_32K_N)
- net ENC_A: now also U301.6 (GPIO3/ADC1_CH3); no longer U301.25 (IO19)
- net ENC_B: now also U301.5 (GPIO2/ADC1_CH2); no longer U301.26 (IO20)
- net ENC_SW_N: now also U301.15 (MTCK/GPIO6/ADC1_CH6); no longer U301.27 (IO21)
- net LED_ACT: now also U301.25 (GPIO19); no longer U301.24 (IO18)
- net LED_FAULT_N: no longer U301.6 (IO3)
- net LED_PWR_EN: now also U301.10 (MTDI/GPIO5/ADC1_CH5); no longer U301.5 (IO2)
- net MCU_LDATA: now reaches U301.16 (MTDO/GPIO7)
- net I2C_SCK renamed LED_ISENSE
- net LED_DATA: no longer names the net of U301.28 (GPIO22)
- no-connect marks 12 -> 13
Other:
- note added: "Note: C303 is marked NRND, but 2M parts still at basic price at jlc"
- note added: "Supply requirement: dedicated USB-C 5 V / 3 A. R307 / R308 provide Rd. No PD negotiation or current detection."
- note removed: "Note: C203 is marked NRND, but 2M parts still at basic price at jlc"
- note removed: "Supply requirement: dedicated USB-C 5 V / 3 A. R206 / R207 provide Rd. No PD negotiation or current detection."
- moved on the sheet: R302

Commit message: Updated silkscreen and production files
Parts:
- C301: LCSC Part # C52923 -> C14445; Rating 25V -> 10V
- D301: JLC_PART E -> B; LCSC Part # C2994781 -> C965804
Changed lines of the file:
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@@
 			)
 		)
-		(property "Rating" "25V"
+		(property "Rating" "10V"
 			(at 38.862 185.674 0)
 			(show_name no)
@@
 			)
 		)
-		(property "LCSC Part #" "C52923"
+		(property "LCSC Part #" "C14445"
 			(at 31.75 182.88 0)
 			(hide yes)
@@
 			)
 		)
-		(property "Datasheet" "https://www.everlighteurope.com/custom/files/datasheets/DSE-0006814.pdf"
+		(property "Datasheet" "https://www.lcsc.com/product-detail/C965804.html"
 			(at 64.77 165.1 0)
 			(hide yes)
@@
 			)
 		)
-		(property "LCSC Part #" "C2994781"
+		(property "LCSC Part #" "C965804"
 			(at 64.77 165.1 0)
 			(hide yes)
@@
 			)
 		)
-		(property "JLC_PART" "E"
+		(property "JLC_PART" "B"
 			(at 64.77 165.1 90)
 			(hide yes)
