File: hardware/power.kicad_sch (KiCad schematic)
At the start: 8 parts, among them U301 TPS62A01ADRL

Commit message: feat: Added led controller sheet
Parts:
- R208: renamed from R301; value 44k8 -> 100k; JLC_PART E -> B; LCSC Part # C852792 -> C25741; TYPE 0.1% -> 1%
- R209: renamed from R302; value 10k -> 22k; JLC_PART E -> B; LCSC Part # C190095 -> C25768; TYPE 0.1% -> 1%
- renumbered C301 to C205, C302 to C206, D301 to D201, L301 to L201, R303 to R211, U301 to U203
Other:
- note added: "* Vin=5V USB-C * Iout(MAX)=1A; share USB budget with LEDs * f(sw)=2.4MHz"
- note added: "R301 / R302: Basic 1% parts. VOUT = 0.6 x (1 + 100k / 22k) = 3.327 V nominal."
- note removed: "* Vin(MAX)=5V * Iout(MAX)=1A, real 500mA from USB-C * f(sw)=2.4MHz"
- title: (none) -> LED power and controls
Changed lines of the file:
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@@
 	(paper "A4")
 	(title_block
+		(title "LED power and controls")
 		(rev "1")
-		(comment 1 "Design for JLCPCB Service")
-	)
-	(text "* Vin(MAX)=5V\n* Iout(MAX)=1A, real 500mA from  USB-C\n* f(sw)=2.4MHz"
+		(comment 1 "JLCPCB")
+	)
+	(text "* Vin=5V USB-C\n* Iout(MAX)=1A; share USB budget with LEDs\n* f(sw)=2.4MHz"
 		(exclude_from_sim no)
 		(at 46.99 45.72 0)
@@
 			)
 			(justify left bottom)
+		)
+	)
+	(text "R301 / R302: Basic 1% parts.\nVOUT = 0.6 x (1 + 100k / 22k) = 3.327 V nominal."
+		(exclude_from_sim no)
+		(at 99.06 106.68 0)
+		(effects
+			(font
+				(size 1.27 1.27)
+			)
+			(justify left top)
 		)
 	)
@@
 		(in_pos_files yes)
 		(dnp no)
-		(property "Reference" "C302"
+		(property "Reference" "C206"
 			(at 127 74.422 0)
 			(show_name no)
@@
 			(project "solar-controller"
 				(path "/1ebd2a79-85df-49b0-bc4d-96f69f4cf347/60d9d9f3-ef40-41c3-9178-d3763959339b"
-					(reference "C302")
+					(reference "C206")
 					(unit 1)
 				)
@@
 		(in_pos_files yes)
 		(dnp no)
-		(property "Reference" "#PWR0307"
+		(property "Reference" "#PWR0222"
 			(at 138.43 64.77 0)
 			(hide yes)
@@
 			(project "solar-controller"
 				(path "/1ebd2a79-85df-49b0-bc4d-96f69f4cf347/60d9d9f3-ef40-41c3-9178-d3763959339b"
-					(reference "#PWR0307")
+					(reference "#PWR0222")
 					(unit 1)
 				)
@@
 		(in_pos_files yes)
 		(dnp no)
-		(property "Reference" "#PWR0304"
+		(property "Reference" "#PWR0219"
 			(at 91.44 74.93 0)
 			(hide yes)
@@
 			(project "solar-controller"
 				(path "/1ebd2a79-85df-49b0-bc4d-96f69f4cf347/60d9d9f3-ef40-41c3-9178-d3763959339b"
-					(reference "#PWR0304")
+					(reference "#PWR0219")
 					(unit 1)
 				)
@@
 		(in_pos_files yes)
 		(dnp no)
-		(property "Reference" "#PWR0302"
+		(property "Reference" "#PWR0217"
 			(at 60.96 90.17 0)
 			(hide yes)
@@
 			(project "solar-controller"
 				(path "/1ebd2a79-85df-49b0-bc4d-96f69f4cf347/60d9d9f3-ef40-41c3-9178-d3763959339b"
-					(reference "#PWR0302")
+					(reference "#PWR0217")
 					(unit 1)
 				)
@@
 		(in_pos_files yes)
 		(dnp no)
-		(property "Reference" "R302"
+		(property "Reference" "R209"
 			(at 117.856 79.502 0)
 			(show_name no)
@@
 			)
 		)
-		(property "Value" "10k"
+		(property "Value" "22k"
 			(at 117.602 81.28 0)
 			(show_name no)
@@
 			)
 		)
-		(property "LCSC Part #" "C190095"
+		(property "LCSC Part #" "C25768"
 			(at 110.49 81.28 0)
 			(hide yes)
@@
 			)
 		)
-		(property "TYPE" "0.1%"
+		(property "TYPE" "1%"
 			(at 115.57 84.836 0)
 			(show_name no)
@@
 			)
 		)
-		(property "JLC_PART" "E"
+		(property "JLC_PART" "B"
 			(at 110.49 81.28 0)
 			(hide yes)
@@
 			(project "solar-controller"
 				(path "/1ebd2a79-85df-49b0-bc4d-96f69f4cf347/60d9d9f3-ef40-41c3-9178-d3763959339b"
-					(reference "R302")
+					(reference "R209")
 					(unit 1)
 				)
@@
 		(in_pos_files yes)
 		(dnp no)
-		(property "Reference" "#PWR0305"
+		(property "Reference" "#PWR0220"
 			(at 110.49 91.44 0)
 			(hide yes)
@@
 			(project "solar-controller"
 				(path "/1ebd2a79-85df-49b0-bc4d-96f69f4cf347/60d9d9f3-ef40-41c3-9178-d3763959339b"
-					(reference "#PWR0305")
+					(reference "#PWR0220")
 					(unit 1)
 				)
@@
 		(dnp no)
 		(fields_autoplaced yes)
-		(property "Reference" "U301"
+		(property "Reference" "U203"
 			(at 82.55 54.61 0)
 			(show_name no)
@@
 			(project "solar-controller"
 				(path "/1ebd2a79-85df-49b0-bc4d-96f69f4cf347/60d9d9f3-ef40-41c3-9178-d3763959339b"
-					(reference "U301")
+					(reference "U203")
 					(unit 1)
 				)
@@
 		(in_pos_files yes)
 		(dnp no)
-		(property "Reference" "#PWR0308"
+		(property "Reference" "#PWR0223"
 			(at 138.43 91.44 0)
 			(hide yes)
@@
 			(project "solar-controller"
 				(path "/1ebd2a79-85df-49b0-bc4d-96f69f4cf347/60d9d9f3-ef40-41c3-9178-d3763959339b"
-					(reference "#PWR0308")
+					(reference "#PWR0223")
 					(unit 1)
 				)
@@
 		(in_pos_files yes)
 		(dnp no)
-		(property "Reference" "#FLG0301"
+		(property "Reference" "#FLG0203"
 			(at 140.335 62.23 0)
 			(hide yes)
@@
 			(project "solar-controller"
 				(path "/1ebd2a79-85df-49b0-bc4d-96f69f4cf347/60d9d9f3-ef40-41c3-9178-d3763959339b"
-					(reference "#FLG0301")
+					(reference "#FLG0203")
 					(unit 1)
 				)
@@
 		(in_pos_files yes)
 		(dnp no)
-		(property "Reference" "#PWR0306"
+		(property "Reference" "#PWR0221"
 			(at 129.54 91.44 0)
 			(hide yes)
@@
 			(project "solar-controller"
 				(path "/1ebd2a79-85df-49b0-bc4d-96f69f4cf347/60d9d9f3-ef40-41c3-9178-d3763959339b"
-					(reference "#PWR0306")
+					(reference "#PWR0221")
 					(unit 1)
 				)
@@
 		(in_pos_files yes)
 		(dnp no)
-		(property "Reference" "R301"
+		(property "Reference" "R208"
 			(at 117.856 68.072 0)
 			(show_name no)
@@
 			)
 		)
-		(property "Value" "44k8"
+		(property "Value" "100k"
 			(at 117.602 69.85 0)
 			(show_name no)
@@
 			)
 		)
-		(property "LCSC Part #" "C852792"
+		(property "LCSC Part #" "C25741"
 			(at 110.49 69.85 0)
 			(hide yes)
@@
 			)
 		)
-		(property "TYPE" "0.1%"
+		(property "TYPE" "1%"
 			(at 115.57 73.406 0)
 			(show_name no)
@@
 			)
 		)
-		(property "JLC_PART" "E"
+		(property "JLC_PART" "B"
 			(at 110.49 69.85 0)
 			(hide yes)
@@
 			(project "solar-controller"
 				(path "/1ebd2a79-85df-49b0-bc4d-96f69f4cf347/60d9d9f3-ef40-41c3-9178-d3763959339b"
-					(reference "R301")
+					(reference "R208")
 					(unit 1)
 				)
@@
 		(in_pos_files yes)
 		(dnp no)
-		(property "Reference" "C301"
+		(property "Reference" "C205"
 			(at 63.754 73.152 0)
 			(show_name no)
@@
 			(project "solar-controller"
 				(path "/1ebd2a79-85df-49b0-bc4d-96f69f4cf347/60d9d9f3-ef40-41c3-9178-d3763959339b"
-					(reference "C301")
+					(reference "C205")
 					(unit 1)
 				)
@@
 		(in_pos_files yes)
 		(dnp no)
-		(property "Reference" "#PWR0303"
+		(property "Reference" "#PWR0218"
 			(at 82.55 82.55 0)
 			(hide yes)
@@
 			(project "solar-controller"
 				(path "/1ebd2a79-85df-49b0-bc4d-96f69f4cf347/60d9d9f3-ef40-41c3-9178-d3763959339b"
-					(reference "#PWR0303")
+					(reference "#PWR0218")
 					(unit 1)
 				)
@@
 		(in_pos_files yes)
 		(dnp no)
-		(property "Reference" "D301"
+		(property "Reference" "D201"
 			(at 144.526 69.85 90)
 			(show_name no)
@@
 			(project "solar-controller"
 				(path "/1ebd2a79-85df-49b0-bc4d-96f69f4cf347/60d9d9f3-ef40-41c3-9178-d3763959339b"
-					(reference "D301")
+					(reference "D201")
 					(unit 1)
 				)
@@
 		(in_pos_files yes)
 		(dnp no)
-		(property "Reference" "L301"
+		(property "Reference" "L201"
 			(at 100.33 57.15 90)
 			(show_name no)
@@
 			(project "solar-controller"
 				(path "/1ebd2a79-85df-49b0-bc4d-96f69f4cf347/60d9d9f3-ef40-41c3-9178-d3763959339b"
-					(reference "L301")
+					(reference "L201")
 					(unit 1)
 				)
@@
 		(dnp no)
 		(fields_autoplaced yes)
-		(property "Reference" "#PWR0301"
+		(property "Reference" "#PWR0216"
 			(at 55.88 64.77 0)
 			(hide yes)
@@
 			(project "solar-controller"
 				(path "/1ebd2a79-85df-49b0-bc4d-96f69f4cf347/60d9d9f3-ef40-41c3-9178-d3763959339b"
-					(reference "#PWR0301")
+					(reference "#PWR0216")
 					(unit 1)
 				)
@@
 		(in_pos_files yes)
 		(dnp no)
-		(property "Reference" "R303"
+		(property "Reference" "R211"
 			(at 145.288 79.502 0)
 			(show_name no)
@@
 			(project "solar-controller"
 				(path "/1ebd2a79-85df-49b0-bc4d-96f69f4cf347/60d9d9f3-ef40-41c3-9178-d3763959339b"
-					(reference "R303")
+					(reference "R211")
 					(unit 1)
 				)

Commit message: feat: WIP pcb layout
Other:
- note added: "Note: C206 is marked NRND, but 2M parts still at basic price at jlc"
- note added: "R208 / R209: Basic 1% parts. VOUT = 0.6 x (1 + 100k / 22k) = 3.327 V nominal."
- note removed: "Note: C302 is marked NRND, but 2M parts still at basic price at jlc"
- note removed: "R301 / R302: Basic 1% parts. VOUT = 0.6 x (1 + 100k / 22k) = 3.327 V nominal."
Changed lines of the file:
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@@
 		)
 	)
-	(text "Note:  C302 is marked NRND, \n       but 2M parts still at basic price at jlc"
+	(text "Note:  C206 is marked NRND, \n       but 2M parts still at basic price at jlc"
 		(exclude_from_sim no)
 		(at 117.602 93.218 0)
@@
 		)
 	)
-	(text "R301 / R302: Basic 1% parts.\nVOUT = 0.6 x (1 + 100k / 22k) = 3.327 V nominal."
+	(text "R208 / R209: Basic 1% parts.\nVOUT = 0.6 x (1 + 100k / 22k) = 3.327 V nominal."
 		(exclude_from_sim no)
 		(at 99.06 106.68 0)

Commit message: Updated silkscreen and production files
Parts:
- D201: JLC_PART E -> B; LCSC Part # C2994781 -> C965804
Changed lines of the file:
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@@
 			)
 		)
-		(property "Datasheet" "https://www.everlighteurope.com/custom/files/datasheets/DSE-0006814.pdf"
+		(property "Datasheet" "https://www.lcsc.com/product-detail/C965804.html"
 			(at 138.43 71.12 0)
 			(hide yes)
@@
 			)
 		)
-		(property "LCSC Part #" "C2994781"
+		(property "LCSC Part #" "C965804"
 			(at 138.43 71.12 0)
 			(hide yes)
@@
 			)
 		)
-		(property "JLC_PART" "E"
+		(property "JLC_PART" "B"
 			(at 138.43 71.12 90)
 			(hide yes)
