File: hardware/solar-controller.kicad_pcb (KiCad board)
At the start: 4 copper layers, 0 parts

Commit message: feat: WIP pcb layout
Parts:
- added C205: 4u7, Capacitor_SMD:C_0805_2012Metric, F.Cu at (111.2, 113.8)
- added C206: 22u, Capacitor_SMD:C_0805_2012Metric, F.Cu at (106.8, 113.8)
- added C301: 1u, Capacitor_SMD:C_0402_1005Metric, F.Cu at (123.1, 99.8)
- added C302: 100n, Capacitor_SMD:C_0402_1005Metric, F.Cu at (133.4, 100.7)
- added C303: 22u, Capacitor_SMD:C_0805_2012Metric, F.Cu at (133.8, 99.1)
- added C304: 100n, Capacitor_SMD:C_0402_1005Metric, F.Cu at (121.8, 118.2)
- added C401: 100n, Capacitor_SMD:C_0402_1005Metric, F.Cu at (118.3, 104.5)
- added C402: 100n, Capacitor_SMD:C_0402_1005Metric, F.Cu at (121.2, 76.4)
- added C403: 100n, Capacitor_SMD:C_0402_1005Metric, F.Cu at (123.3, 73.5)
- added C404: 470u, Capacitor_SMD:CP_Elec_6.3x7.7, F.Cu at (132.6, 75.9)
- added C405: 22u, Capacitor_SMD:C_0805_2012Metric, F.Cu at (123.5, 77.8)
- added C407: 100n, Capacitor_SMD:C_0402_1005Metric, F.Cu at (115.6, 106.2)
- added C408: 100n, Capacitor_SMD:C_0402_1005Metric, F.Cu at (123.7, 103.0)
- added D201: LED_GREEN, LED_SMD:LED_0603_1608Metric, F.Cu at (103.8, 114.1)
- added D301: LED_ACT, LED_SMD:LED_0603_1608Metric, F.Cu at (126.8, 127.7)
- added D401: SS34, Diode_SMD:D_SMA, F.Cu at (127.6, 68.4)
- added H1: M2.5, MountingHole:MountingHole_2.7mm_M2.5, F.Cu at (103.5, 126.5)
- added H2: M2.5, MountingHole:MountingHole_2.7mm_M2.5, F.Cu at (134.5, 126.5)
- added H3: M2.5, MountingHole:MountingHole_2.7mm_M2.5, F.Cu at (103.5, 63.5)
- added H4: M2.5, MountingHole:MountingHole_2.7mm_M2.5, F.Cu at (134.5, 63.5)
- added J301: USB_C_Receptacle_USB2.0, Connector_USB:USB_C_Receptacle_HRO_TYPE-C-31-M-12, F.Cu at (119.0, 127.3)
- added J401: ZX-XH2.54-3PWT, SolarController:Megastar_ZX-XH2.54-3PWT, F.Cu at (119.0, 69.8)
- added L201: 1u, Inductor_SMD:L_1008_2520Metric, F.Cu at (109.0, 117.0)
- added R208: 100k, Resistor_SMD:R_0402_1005Metric, F.Cu at (108.5, 112.0)
- added R209: 22k, Resistor_SMD:R_0402_1005Metric, F.Cu at (109.6, 112.0)
- added R211: 2k2, Resistor_SMD:R_0402_1005Metric, F.Cu at (103.5, 116.3)
- added R301: 10k, Resistor_SMD:R_0402_1005Metric, F.Cu at (124.2, 99.8)
- added R302: 10k, Resistor_SMD:R_0402_1005Metric, F.Cu at (124.2, 111.8)
- added R303: 10k, Resistor_SMD:R_0402_1005Metric, F.Cu at (125.8, 119.1)
- added R306: 2k2, Resistor_SMD:R_0402_1005Metric, F.Cu at (128.2, 128.0)
- added R307: 5k1, Resistor_SMD:R_0402_1005Metric, F.Cu at (113.1, 123.0)
- added R308: 5k1, Resistor_SMD:R_0402_1005Metric, F.Cu at (124.9, 123.0)
- added R403: 1k, Resistor_SMD:R_0402_1005Metric, F.Cu at (125.4, 74.4)
- added R404: 10k, Resistor_SMD:R_0402_1005Metric, F.Cu at (123.7, 104.1)
- added R405: 2k2, Resistor_SMD:R_0402_1005Metric, F.Cu at (130.0, 71.0)
- added R406: 2k2, Resistor_SMD:R_0402_1005Metric, F.Cu at (120.1, 75.5)
- added R407: 100k, Resistor_SMD:R_0402_1005Metric, F.Cu at (121.2, 74.4)
- added R408: 10k, Resistor_SMD:R_0402_1005Metric, F.Cu at (117.8, 101.8)
- added R409: 330, Resistor_SMD:R_0402_1005Metric, F.Cu at (112.9, 102.3)
- added R410: 100k, Resistor_SMD:R_0402_1005Metric, F.Cu at (111.8, 102.3)
- added R411: 2k2, Resistor_SMD:R_0402_1005Metric, F.Cu at (129.4, 91.0)
- added R412: 2k2, Resistor_SMD:R_0402_1005Metric, F.Cu at (129.4, 86.0)
- added R413: 10k, Resistor_SMD:R_0402_1005Metric, F.Cu at (108.5, 91.0)
- added R414: 100k, Resistor_SMD:R_0402_1005Metric, F.Cu at (126.5, 74.4)
- added SW301: RESET, Button_Switch_SMD:SW_SPST_TS-1088-xR020, F.Cu at (127.8, 99.3)
- added SW302: BOOT, Button_Switch_SMD:SW_SPST_TS-1088-xR020, F.Cu at (127.8, 116.8)
- added SW402: EC11J1525402, SolarController:ALPS_EC11J1525402, F.Cu at (119.0, 88.0)
- added U203: TPS62A01ADRL, Package_TO_SOT_SMD:SOT-563, F.Cu at (109.0, 114.3)
- added U301: ESP32-C6-MINI-1U-H4, PCM_Espressif:ESP32-C6-MINI-1U, F.Cu at (133.3, 108.1)
- added U302: USBLC6-2SC6, Package_TO_SOT_SMD:SOT-23-6, F.Cu at (119.5, 118.2)
- added U402: TPS259531DSGR, Package_SON:Texas_DSG0008A_WSON-8-1EP_2x2mm_P0.5mm_EP0.9x1.6mm, F.Cu at (123.3, 75.4)
- added U403: SN74LVC1T45DBVR, Package_TO_SOT_SMD:SOT-23-6, F.Cu at (115.6, 103.9)
Routing:
- net /[3] MCU/USB_D-: track 0.00 -> 15.8 mm
- net /[3] MCU/USB_D+: track 0.00 -> 15.2 mm
- net +3V3: track 0.00 -> 10.6 mm, vias 0 -> 1
- net /[3] MCU/USB_CONN_CC1: track 0.00 -> 9.16 mm
- net /[3] MCU/USB_CONN_CC2: track 0.00 -> 8.55 mm
- net /[3] MCU/USB_CONN_D+: track 0.00 -> 7.28 mm
- net /[3] MCU/RESET: track 0.00 -> 6.21 mm
- net /[3] MCU/USB_CONN_D-: track 0.00 -> 6.14 mm
- net /[2] Power/SW: track 0.00 -> 3.06 mm
- net /[2] Power/FB: track 0.00 -> 2.43 mm
- net /[4] LED control/ILM: track 0.00 -> 2.36 mm
- net Net-(D201-K): track 0.00 -> 1.55 mm
- net /[3] MCU/IO8: track 0.00 -> 1.50 mm
- net VBUS: track 0.00 -> 1.42 mm
- net GND: vias 0 -> 1
- added copper zone on F.Cu, net +3V3
- added copper zone on F.Cu, net +5V
- added copper zone on B.Cu, net GND
- added copper zone on F.Cu, net GND
- added copper zone on F.Cu, net VBUS
Other:
- board outline added: 38 x 70 mm
- copper layers 4 -> 2
- board text added: "3.3V"
- board text added: "4x M2.5 screws through PCB into shell posts (Ø6 dashed)"
- board text added: "Bottom shell: Ø6 support post under encoder, no B-side parts"
- board text added: "ESP32-C6-MINI-1U: no PCB antenna, U.FL socket left unused"
- board text added: "Enclosure (User.Drawings): 44 x 90 x ~22 mm, 2 mm walls"
- board text added: "Encoder axis 42 from USB edge = enclosure centre"
- board text added: "Lid hole >= Ø10, knob Ø23 with 2 mm gap above lid"
- board text added: "PCB 38 x 70 mm, 1.6 mm, 4 layers, corners R3"
- board text added: "PCB sits 1 mm from USB-end wall, 1 mm side clearance"
- board text added: "USB-C shell front 1 mm past PCB edge = flush with inner wall"
- board text added: "USB-C, encoder and LED connector on centre line x = 19"
- board text added: "cable clamp zone"
- board text added: "inner wall"
- board text added: "knob Ø23"

Commit message: Updated silkscreen and production files
Parts:
- removed H1, H2, H3, H4: M2.5, MountingHole:MountingHole_2.7mm_M2.5
- added G***: LOGO, LOGO, F.Cu at (113.4, 104.9)
- added H101: GND, MountingHole:MountingHole_2.7mm_M2.5_ISO14580_Pad, F.Cu at (103.5, 126.5)
- added H102: GND, MountingHole:MountingHole_2.7mm_M2.5_ISO14580_Pad, F.Cu at (134.5, 126.5)
- added H103: GND, MountingHole:MountingHole_2.7mm_M2.5_ISO14580_Pad, F.Cu at (134.5, 63.5)
- added H104: GND, MountingHole:MountingHole_2.7mm_M2.5_ISO14580_Pad, F.Cu at (103.5, 63.5)
- moved C407 30.7 mm to (115.0, 75.5), turned to 90 degrees
- moved R410 29.8 mm to (113.4, 72.5), turned to 180 degrees
- moved C401 29.4 mm to (109.7, 76.4), turned to -90 degrees
- moved R409 28.7 mm to (113.4, 73.6), turned to 0 degrees
- moved U403 27.2 mm to (112.4, 76.9), turned to 0 degrees
- moved R408 24.8 mm to (109.7, 78.4), turned to -90 degrees
- moved R405 11.5 mm to (120.4, 77.2), turned to 180 degrees
- moved R406 11.2 mm to (131.1, 77.8)
- moved D401 10.0 mm to (120.0, 74.9), turned to 180 degrees
- moved R407 9.41 mm to (129.9, 77.8), turned to -90 degrees
- moved C402 8.77 mm to (129.9, 75.8), turned to 90 degrees
- moved C403 6.95 mm to (127.8, 78.8), turned to 180 degrees
- moved C404 6.67 mm to (130.4, 69.6)
- moved C405 5.33 mm to (127.7, 74.5), turned to 0 degrees
- moved C301 4.80 mm to (127.7, 98.4), turned to 0 degrees
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Routing:
- net VBUS: track 1.42 -> 116.7 mm, vias 0 -> 8
- net /[3] MCU/MCU_LDATA: track 0.00 -> 51.9 mm
- net /[3] MCU/LED_FAULT_N: track 0.00 -> 38.7 mm
- net /[3] MCU/ENC_SW_N: track 0.00 -> 32.6 mm
- net /[3] MCU/LED_PWR_EN: track 0.00 -> 31.5 mm
- net /[3] MCU/LED_ISENSE: track 0.00 -> 28.1 mm
- net /[3] MCU/ENC_B: track 0.00 -> 23.1 mm
- net /[3] MCU/ENC_A: track 0.00 -> 17.6 mm
- net /[4] LED control/CONN_LDATA: track 0.00 -> 13.7 mm
- net /[3] MCU/LED_ACT: track 0.00 -> 12.3 mm
- net +3V3: track 10.6 -> 22.7 mm, vias 1 -> 20
- net +5V: track 0.00 -> 10.5 mm
- net /[3] MCU/BOOT: track 0.00 -> 8.01 mm
- net /[4] LED control/B_LDATA: track 0.00 -> 5.47 mm
- net /[3] MCU/RESET: track 6.21 -> 9.76 mm
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- added copper zone on In2.Cu, net +3V3
- added copper zone on In1.Cu, net GND
Other:
- copper layers 2 -> 4
- board text added: "5V"
- board text added: "ACT"
- board text added: "BOOT"
- board text added: "DATA"
- board text added: "GND"
- board text added: "RESET"
